Commit message: add the room map, gamepad_telelop using joy for modern controllers and odom topic

File: src/motor_control/description/car.urdf (robot description, URDF)
Before this commit: robot hiwonder_ackermann, 8 links, 7 joints
Links:
- removed link laser_link
- added link laser; visual cylinder length=0.02 radius=0.035
Joints:
- joint laser_joint: child laser_link -> laser; origin xyz=0.175 0.0 0.07 rpy=0 0 3.14159 -> xyz=0.175 0.0 0.092 rpy=0 0 3.14159
